Commit message: Added IMU sensor

File: steer_bot_description/urdf/steer_bot.urdf.xacro (robot description, xacro)
@@ -138,3 +138,56 @@
     <material>Gazebo/Green</material>
   </gazebo>
+<!-- IMU -->
+  <!-- Imu -->
+  <xacro:property name="imu_xsize" value="0.05" />
+  <xacro:property name="imu_ysize" value="0.05" />
+  <xacro:property name="imu_zsize" value="0.05" />
+  <xacro:property name="imu_mass"  value="0.1" />
+  <xacro:property name="imu_xpos"  value="0" />
+  <xacro:property name="imu_ypos"  value="0.00" />
+  <xacro:property name="imu_zpos"  value="${base_height/2}" />
+  <!-- Imu -->
+  <link name="imu_box" >
+    <visual>
+      <!--material name="blue" /-->  <!--Funziona per Rviz non per Gazebo-->
+      <geometry>
+        <box size="${imu_xsize} ${imu_ysize} ${imu_zsize}" />
+      </geometry>
+    </visual>
+    <collision>
+      <geometry>
+        <box size="${imu_xsize} ${imu_ysize} ${imu_zsize}" />
+      </geometry>
+    </collision>
+    <xacro:solid_cuboid_inertial
+        rpy="0 0 0" xyz="${imu_xsize} ${imu_ysize} ${imu_zsize}"
+        mass="${imu_mass}"
+        x="${imu_xpos}" y="${imu_ypos}" z="${imu_zpos}" />
+  </link>
+  <joint name="joint_imu_box" type="fixed">
+    <origin xyz="${imu_xpos} ${imu_ypos} ${imu_zpos}" rpy="0 0 0" />
+    <parent link="base_link" />
+    <child link="imu_box" />
+  </joint>
+  <gazebo reference="imu_box">
+    <material>Gazebo/White</material> <!--Funziona per Rviz non per Gazebo-->
+    <gravity>true</gravity>
+    <sensor name="imu_sensor" type="imu">
+      <always_on>true</always_on>
+      <update_rate>100</update_rate>
+      <visualize>true</visualize>
+      <topic>__default_topic__</topic>
+      <plugin filename="libgazebo_ros_imu_sensor.so" name="imu_plugin" >
+        <topicName>imu</topicName>
+        <bodyName>imu_link</bodyName>
+        <updateRateHZ>10.0</updateRateHZ>
+        <gaussianNoise>0.0</gaussianNoise>
+        <xyzOffset>0 0 0</xyzOffset>
+        <rpyOffset>0 0 0</rpyOffset>
+        <frameName>imu_link</frameName>
+        <inertialOrientationAsReference>false</inertialOrientationAsReference>
+      </plugin>
+      <pose>0 0 0 0 0 0</pose>
+    </sensor>
+  </gazebo>
 </robot>

Commit message: Edit dimensions

File: steer_bot_description/urdf/steer_bot.urdf.xacro (robot description, xacro)
@@ -42,11 +42,11 @@
   <xacro:property name="deg_to_rad" value="0.01745329251994329577"/>
   <!-- Robot base dimensions -->
-  <xacro:property name="base_length" value="0.5" />
-  <xacro:property name="base_width" value="0.3" />
-  <xacro:property name="base_height" value="0.1" />
-  <xacro:property name="base_mass" value="5" />
+  <xacro:property name="base_length" value="0.37" />
+  <xacro:property name="base_width" value="0.14" />
+  <xacro:property name="base_height" value="0.07" />
+  <xacro:property name="base_mass" value="0.07" />
   <!-- Wheel link dimensions -->
-  <xacro:property name="wheel_radius" value="0.1" />
-  <xacro:property name="wheel_thickness" value="0.08" />
+  <xacro:property name="wheel_radius" value="0.04" />
+  <xacro:property name="wheel_thickness" value="0.015" />
   <xacro:property name="wheel_mass" value="1" />
   <!-- Steering link dimensions -->

Commit message: revert to previous status

File: steer_bot_description/urdf/steer_bot.urdf.xacro (robot description, xacro)
@@ -42,11 +42,11 @@
   <xacro:property name="deg_to_rad" value="0.01745329251994329577"/>
   <!-- Robot base dimensions -->
-  <xacro:property name="base_length" value="0.37" />
-  <xacro:property name="base_width" value="0.14" />
-  <xacro:property name="base_height" value="0.07" />
-  <xacro:property name="base_mass" value="0.07" />
+  <xacro:property name="base_length" value="0.5" />
+  <xacro:property name="base_width" value="0.3" />
+  <xacro:property name="base_height" value="0.1" />
+  <xacro:property name="base_mass" value="5" />
   <!-- Wheel link dimensions -->
-  <xacro:property name="wheel_radius" value="0.04" />
-  <xacro:property name="wheel_thickness" value="0.015" />
+  <xacro:property name="wheel_radius" value="0.1" />
+  <xacro:property name="wheel_thickness" value="0.08" />
   <xacro:property name="wheel_mass" value="1" />
   <!-- Steering link dimensions -->

Commit message: Infrastructure for drawing odometry

File: steer_bot_description/urdf/steer_bot.urdf.xacro (robot description, xacro)
@@ -27,5 +27,5 @@
       <legacyModeNS>false</legacyModeNS>
     </plugin>
-<!--    <plugin name="p3d_base_controller" filename="libgazebo_ros_p3d.so">
+    <plugin name="p3d_base_controller" filename="libgazebo_ros_p3d.so">
       <alwaysOn>true</alwaysOn>
       <updateRate>50.0</updateRate>
@@ -33,9 +33,8 @@
       <topicName>pose_ground_truth</topicName>
       <gaussianNoise>0.00</gaussianNoise>
-      <frameName>odom</frameName>
+      <frameName>world</frameName>
       <xyzOffsets>0 0 0</xyzOffsets>
       <rpyOffsets>0 0 0</rpyOffsets>
     </plugin>
--->
   </gazebo>
   <!-- Math constants -->
@@ -161,5 +160,5 @@
   <link name="imu_box" >
     <visual>
-      <!--material name="blue" /-->  <!--Funziona per Rviz non per Gazebo-->
+      <material name="blue" />
       <geometry>
         <box size="${imu_xsize} ${imu_ysize} ${imu_zsize}" />
@@ -182,5 +181,5 @@
   </joint>
   <gazebo reference="imu_box">
-    <material>Gazebo/White</material> <!--Funziona per Rviz non per Gazebo-->
+    <material>Gazebo/White</material>
     <gravity>true</gravity>
     <sensor name="imu_sensor" type="imu">
@@ -193,5 +192,5 @@
         <bodyName>imu_link</bodyName>
         <updateRateHZ>10.0</updateRateHZ>
-        <gaussianNoise>0.0</gaussianNoise>
+        <gaussianNoise>2.89e-08</gaussianNoise>
         <xyzOffset>0 0 0</xyzOffset>
         <rpyOffset>0 0 0</rpyOffset>

Commit message: Added chronometer and camera

File: steer_bot_description/urdf/steer_bot.urdf.xacro (robot description, xacro)
@@ -148,4 +148,76 @@
     <material>Gazebo/Green</material>
   </gazebo>
+<!-- CAMERA -->
+<xacro:property name="camera_dim" value="0.05" /> <!-- Size of square 'camera' box -->
+<xacro:property name="camera_xpos"  value="-0.1" />
+<xacro:property name="camera_ypos"  value="0" />
+<xacro:property name="camera_zpos"  value="${base_height/2 + 0.12}" />
+ <joint name="camera_joint" type="fixed">
+    <axis xyz="0 1 0" />
+    <origin xyz="${camera_xpos} ${camera_ypos} ${camera_zpos}" rpy="0 0 0"/>
+    <parent link="base_link"/>
+    <child link="camera_link"/>
+  </joint>
+  <!-- Camera -->
+  <link name="camera_link">
+    <collision>
+      <origin xyz="0 0 0" rpy="0 0 0"/>
+      <geometry>
+    <box size="${camera_dim} ${camera_dim} ${camera_dim}"/>
+      </geometry>
+    </collision>
+    <visual>
+      <origin xyz="0 0 0" rpy="0 0 0"/>
+      <geometry>
+    <box size="${camera_dim} ${camera_dim} ${camera_dim}"/>
+      </geometry>
+      <material name="red"/>
+    </visual>
+    <inertial>
+      <mass value="1e-5" />
+      <origin xyz="0 0 0" rpy="0 0 0"/>
+      <inertia ixx="1e-6" ixy="0" ixz="0" iyy="1e-6" iyz="0" izz="1e-6" />
+    </inertial>
+  </link>
+  <!-- camera -->
+  <gazebo reference="camera_link">
+    <sensor type="camera" name="camera1">
+      <update_rate>30.0</update_rate>
+      <camera name="head">
+        <horizontal_fov>1.3962634</horizontal_fov>
+        <image>
+          <width>800</width>
+          <height>800</height>
+          <format>R8G8B8</format>
+        </image>
+        <clip>
+          <near>0.02</near>
+          <far>300</far>
+        </clip>
+        <noise>
+          <type>gaussian</type>
+          <!-- Noise is sampled independently per pixel on each frame.
+               That pixel's noise value is added to each of its color
+               channels, which at that point lie in the range [0,1]. -->
+          <mean>0.0</mean>
+          <stddev>0.007</stddev>
+        </noise>
+      </camera>
+      <plugin name="camera_controller" filename="libgazebo_ros_camera.so">
+        <alwaysOn>true</alwaysOn>
+        <updateRate>0.0</updateRate>
+        <cameraName>rrbot/camera1</cameraName>
+        <imageTopicName>image_raw</imageTopicName>
+        <cameraInfoTopicName>camera_info</cameraInfoTopicName>
+        <frameName>camera_link</frameName>
+        <hackBaseline>0.07</hackBaseline>
+        <distortionK1>0.0</distortionK1>
+        <distortionK2>0.0</distortionK2>
+        <distortionK3>0.0</distortionK3>
+        <distortionT1>0.0</distortionT1>
+        <distortionT2>0.0</distortionT2>
+      </plugin>
+    </sensor>
+  </gazebo>
 <!-- IMU -->
   <!-- Imu -->

Commit message: add_Lidar

File: steer_bot_description/urdf/steer_bot.urdf.xacro (robot description, xacro)
@@ -148,4 +148,67 @@
     <material>Gazebo/Green</material>
   </gazebo>
+<!-- LIDAR -->
+<link name="lidar_link">
+    <collision>
+      <origin xyz="0.5 0 0" rpy="0 0 0"/>
+      <geometry>
+    <box size="0.1 0.1 0.1"/>
+      </geometry>
+    </collision>
+    <visual>
+      <origin xyz="0 0 0" rpy="0 0 0"/>
+      <geometry>
+        <mesh filename="package://steer_bot_description/hokuyo.dae"/>
+      </geometry>
+    </visual>
+    <inertial>
+      <mass value="1e-5" />
+      <origin xyz="0 0 0" rpy="0 0 0"/>
+      <inertia ixx="1e-6" ixy="0" ixz="0" iyy="1e-6" iyz="0" izz="1e-6" />
+    </inertial>
+  </link>
+<joint name="lidar_link_joint" type="fixed">
+    <axis xyz="0.1 1 0" />
+    <origin xyz="0.15 0 0.1" rpy="0 0 0"/>
+    <parent link="base_link"/>
+    <child link="lidar_link"/>
+  </joint>
+   <!-- hokuyo -->
+  <gazebo reference="lidar_link">
+    <sensor type="gpu_ray" name="lidar_sensor">
+      <pose>0 0 0 0 0 0</pose>
+      <visualize>true</visualize>
+      <update_rate>40</update_rate>
+      <ray>
+        <scan>
+          <horizontal>
+            <samples>720</samples>
+            <resolution>1</resolution>
+            <min_angle>-1.570796</min_angle>
+            <max_angle>1.570796</max_angle>
+          </horizontal>
+        </scan>
+        <range>
+          <min>0.10</min>
+          <max>30.0</max>
+          <resolution>0.01</resolution>
+        </range>
+        <noise>
+          <type>gaussian</type>
+          <!-- Noise parameters based on published spec for Hokuyo laser
+               achieving "+-30mm" accuracy at range < 10m.  A mean of 0.0m and
+               stddev of 0.01m will put 99.7% of samples within 0.03m of the true
+               reading. -->
+          <mean>0.0</mean>
+          <stddev>0.01</stddev>
+        </noise>
+      </ray>
+      <plugin name="gazebo_ros_head_hokuyo_controller" filename="libgazebo_ros_gpu_laser.so">
+        <topicName>/rrbot/laser/scan</topicName>
+        <frameName>lidar_link</frameName>
+      </plugin>
+    </sensor>
+  </gazebo>
+<!-- FINE LIDAR -->
 <!-- IMU -->
   <!-- Imu -->

Commit message: spostamento lidar

File: steer_bot_description/urdf/steer_bot.urdf.xacro (robot description, xacro)
@@ -169,6 +169,6 @@
   </link>
 <joint name="lidar_link_joint" type="fixed">
-    <axis xyz="0.1 1 0" />
-    <origin xyz="0.15 0 0.1" rpy="0 0 0"/>
+    <axis xyz="0 0 0" />
+    <origin xyz="0.32 0 -0.01" rpy="0 0 0"/>
     <parent link="base_link"/>
     <child link="lidar_link"/>

Commit message: MOdIFICHE CAMERA

File: steer_bot_description/urdf/steer_bot.urdf.xacro (robot description, xacro)
@@ -211,4 +211,76 @@
   </gazebo>
 <!-- FINE LIDAR -->
+<!-- CAMERA -->
+<xacro:property name="camera_dim" value="0.05" /> <!-- Size of square 'camera' box -->
+<xacro:property name="camera_xpos"  value="-0.1" />
+<xacro:property name="camera_ypos"  value="0" />
+<xacro:property name="camera_zpos"  value="${base_height/2 + 0.12}" />
+ <joint name="camera_joint" type="fixed">
+    <axis xyz="0 1 0" />
+    <origin xyz="${camera_xpos} ${camera_ypos} ${camera_zpos}" rpy="0 0 0"/>
+    <parent link="base_link"/>
+    <child link="camera_link"/>
+  </joint>
+  <!-- Camera -->
+  <link name="camera_link">
+    <collision>
+      <origin xyz="0 0 0" rpy="0 0 0"/>
+      <geometry>
+    <box size="${camera_dim} ${camera_dim} ${camera_dim}"/>
+      </geometry>
+    </collision>
+    <visual>
+      <origin xyz="0 0 0" rpy="0 0 0"/>
+      <geometry>
+    <box size="${camera_dim} ${camera_dim} ${camera_dim}"/>
+      </geometry>
+      <material name="red"/>
+    </visual>
+    <inertial>
+      <mass value="1e-5" />
+      <origin xyz="0 0 0" rpy="0 0 0"/>
+      <inertia ixx="1e-6" ixy="0" ixz="0" iyy="1e-6" iyz="0" izz="1e-6" />
+    </inertial>
+  </link>
+  <!-- camera -->
+  <gazebo reference="camera_link">
+    <sensor type="camera" name="camera1">
+      <update_rate>30.0</update_rate>
+      <camera name="head">
+        <horizontal_fov>1.3962634</horizontal_fov>
+        <image>
+          <width>800</width>
+          <height>800</height>
+          <format>R8G8B8</format>
+        </image>
+        <clip>
+          <near>0.02</near>
+          <far>300</far>
+        </clip>
+        <noise>
+          <type>gaussian</type>
+          <!-- Noise is sampled independently per pixel on each frame.
+               That pixel's noise value is added to each of its color
+               channels, which at that point lie in the range [0,1]. -->
+          <mean>0.0</mean>
+          <stddev>0.007</stddev>
+        </noise>
+      </camera>
+      <plugin name="camera_controller" filename="libgazebo_ros_camera.so">
+        <alwaysOn>true</alwaysOn>
+        <updateRate>0.0</updateRate>
+        <cameraName>rrbot/camera1</cameraName>
+        <imageTopicName>image_raw</imageTopicName>
+        <cameraInfoTopicName>camera_info</cameraInfoTopicName>
+        <frameName>camera_link</frameName>
+        <hackBaseline>0.07</hackBaseline>
+        <distortionK1>0.0</distortionK1>
+        <distortionK2>0.0</distortionK2>
+        <distortionK3>0.0</distortionK3>
+        <distortionT1>0.0</distortionT1>
+        <distortionT2>0.0</distortionT2>
+      </plugin>
+    </sensor>
+  </gazebo>
 <!-- IMU -->
   <!-- Imu -->
